File: fan-controller-pico_hmi.kicad_sch (KiCad schematic)
At the start: 18 parts, among them U4 OLEDM0.96-1YB-I2C

Commit message: tl;dr: switched to 4-layer pcb, overhauled 12vdc rail and protections, added 5vdc ORing ======================================================================== added:   ./       .gitignore - ignore lockfile
------------------------------------------------------------------------
removed:
  licenses/ - switched fonts to all WebPlus_ToshibaSat_8x14 and 9x16
      curie-LICENSE.txt
      curie-NOTICE.txt
      scientifica-LICENSE.txt
      scientifica-NOTICE.txt

------------------------------------------------------------------------
modified:
  ./
      README.md - updated to reflect changes in design
      fan-controller-pico_hmi.kicad_sch - added connector circuit, added
        pico pin connections
      fan-controller-txu0204-pico.kicad_pcb - changed to 4-layer design,
        changed protection circuit designs to use p-fet and polyfuse,
        split 12vdc rail into separate lines for fans and dc-dc
        converter, added lm66200 ORing diode, changed various netclass
        clearances, adjusted positions of tvs diodes for the fans'
        +12vdc pins
      fan-controller-txu0204-pico.kicad_sch - removed efuse, switched to
        p-fet reverse polarity protection, polyfuse for dc-dc converter,
        changed tvs diode for power connector to something more robust,
        added lm66200 ORing dual ideal diode for dc-dc converter 5v
        output and vbus to vsys control
      fan-controller-txu0204-pico.kicad_pro - see above
Parts:
- added CN4: HMI, symbol lib_fan-controller-txu0204-pico:connector_hmi-board-in
- S1: footprint PEC12R-4120F-S0012:XDCR_PEC12R-4120F-S0012 -> lsc-switch:XDCR_PEC12R-4120F-S0012_BOURNS
Connections:
- net 3V3: now also CN4.2 (3V3)
- net 587_CTRL: now also CN4.9 (RGB)
- net ENCODER_A: now also CN4.7 (ECB)
- net ENCODER_B: now also CN4.6 (ECA)
- net GND: now also CN4.1 (GND)
- net I2C_SCL: now also CN4.4 (SCL)
- net I2C_SDA: now also CN4.5 (SDA)
- net PICO_RESET: now also CN4.8 (RST)
- new net VSYS: CN4.3 (VSYS)
- no-connect marks 1 -> 2
