File: fan-controller-txu0204-pico.kicad_sch (KiCad schematic)
At the start: 58 parts, among them CN1 PWR, CN2 RaspberryPi_Pico, CN3 RaspberryPi_Pico, Q1 RU1C002ZP, U1 TPS259472A, U2 TXU0204, U3 TXU0204

Commit message: tl;dr: switched to 4-layer pcb, overhauled 12vdc rail and protections, added 5vdc ORing ======================================================================== added:   ./       .gitignore - ignore lockfile
------------------------------------------------------------------------
removed:
  licenses/ - switched fonts to all WebPlus_ToshibaSat_8x14 and 9x16
      curie-LICENSE.txt
      curie-NOTICE.txt
      scientifica-LICENSE.txt
      scientifica-NOTICE.txt

------------------------------------------------------------------------
modified:
  ./
      README.md - updated to reflect changes in design
      fan-controller-pico_hmi.kicad_sch - added connector circuit, added
        pico pin connections
      fan-controller-txu0204-pico.kicad_pcb - changed to 4-layer design,
        changed protection circuit designs to use p-fet and polyfuse,
        split 12vdc rail into separate lines for fans and dc-dc
        converter, added lm66200 ORing diode, changed various netclass
        clearances, adjusted positions of tvs diodes for the fans'
        +12vdc pins
      fan-controller-txu0204-pico.kicad_sch - removed efuse, switched to
        p-fet reverse polarity protection, polyfuse for dc-dc converter,
        changed tvs diode for power connector to something more robust,
        added lm66200 ORing dual ideal diode for dc-dc converter 5v
        output and vbus to vsys control
      fan-controller-txu0204-pico.kicad_pro - see above
Parts:
- removed C1: 10uF, lsc-capacitors-added:C_GRM18_0603_1608Metric_MURATA, symbol capacitors-added:template-capacitor-ceramic
- removed C2: 0.56nF, lsc-capacitors-added:C_GRM18_0603_1608Metric_MURATA, symbol capacitors-added:template-capacitor-ceramic
- removed D1: TPSMA6L12A, lsc-diode-smd:DIO_DO221AC_TPSMA6LSeries_LTF, symbol tvs-diodes-added:TPSMA6L12A_LITTELFUSE
- removed D4: RBS1MM40A, lsc-diode-smd:CR_RBS1MM_ROM, symbol schottky-diodes-added:RBS1MM40A_ROHM
- removed R1: 470k, lsc-resistor:R_RK37H_0402_1005Metric_KOA, symbol resistors-added:template-resistor-small-us
- removed R2: 97.6k, lsc-resistor:R_RK37H_0402_1005Metric_KOA, symbol resistors-added:template-resistor-small-us
- removed R3: 390k, lsc-resistor:R_RK37H_0402_1005Metric_KOA, symbol resistors-added:template-resistor-small-us
- removed R4: 2.43k, lsc-resistor:R_RK37H_0402_1005Metric_KOA, symbol resistors-added:template-resistor-small-us
- removed R5: 47k, lsc-resistor:R_RK37H_0402_1005Metric_KOA, symbol resistors-added:template-resistor-small-us
- removed R7: 5.5k, lsc-resistor:R_RK37H_0402_1005Metric_KOA, symbol resistors-added:template-resistor-small-us
- removed U1: TPS259472A, lsc-qfn:VFQFN10_RPW0010A_TI, symbol power-protection-added:TPS259472A_TI
- added D1: SMAJ16CA, lsc-diode-smd:DIO_SMB_LOWVOLTAGE_DIODES, symbol tvs-diodes-added:SMAJ16CA_WURTH
- added D4: SGL1-20, lsc-diode-smd:DIO_DO213AA_MINIMELF, symbol schottky-diodes-added:SGL1-20_DIOTEC
- added D5, D6: SMF12A, lsc-diode-smd:D_SOD-123F_EATON, symbol tvs-diodes-added:SMF12A_EATON
- added F1: 2016L150/33DR, lsc-polyfuse:PTS1206_FUSC3216X68N_EATON, symbol polyfuse-added:2016L150/33DR_LITTEL
- added Q2: DMP3014SFDE, lsc-dfn-vdfn-tdfn:TRANS_6-UDFN_U-DFN2020-6-E_DIO, symbol mosfets-p-channel-added:DMP3014SFDE_DIODES
- added R1: 274, lsc-resistor:R_RK37H_0402_1005Metric_KOA, symbol resistors-added:KOA_RK73H1ETTP1000F
- added R9: 5.62k, lsc-resistor:R_RK37H_0402_1005Metric_KOA, symbol resistors-added:template-resistor-small-us
- added U5: LM66200, lsc-standard-chip-carrier:SOT-583_SOT-5X3_DRL0008A_TEX, symbol power-protection-added:LM66200_TI
- added ZD1: MM3Z20B-AQ, lsc-diode-smd:D_SOD-323F_SOD323F_DIODES, symbol zener-diodes-added:MM3Z20B-AQ_DIOTEC
- R11, R12, R15, R16, R17, R18, R23, R24: value 10k -> 750
- R21, R22, R25, R26: value 7.5k -> 750
- U2, U3: Current - Supply (none) -> μA; Interface / Protocol 1 (none) -> VCCA - GPIO; Interface / Protocol 2 (none) -> VCCP - GPIO; Manufacturer (none) -> Texas Instruments; Voltage - Supply (none) -> V
Connections:
- net GPIO2 is gone; now on net PICO_PWM_FAN1: CN2.4 (GPIO2)
- net GPIO3 is gone; now on net PICO_PWM_FAN2: CN2.5 (GPIO3)
- net +12V_UNPROTECTED: now also D1.1 (A1), Q2.1 (DRAIN)
- net GND: now also D1.2 (A2), D4.2 (A), D5.2 (A), D6.2 (A), R1.1, U5.4 (~{ON}), U5.[1,5] (GND)
- net PICO_PWM_FAN1: no longer CN2.6 (GPIO4)
- net PICO_PWM_FAN2: no longer CN2.7 (GPIO5)
- net VBUS: now also U5.3 (VIN1)
- net +12V_PROTECTED renamed +12VDC
- net +12VDC: now also D5.1 (K), D6.1 (K), F1.1, Q2.3 (SOURCE), Q2.4 (SOURCE), ZD1.1 (K); no longer PSU1.1 (IN), R21.2, R22.2, R25.2, R26.2
- net 3V3 renamed +3.3VDC
- net PWRGD renamed LM66200_STAT
- net LM66200_STAT: now also R9.1, U5.8 (ST)
- net VSYS renamed +5VDC
- net +5VDC: now also R21.2, R22.2, R25.2, R26.2, R9.2, U5.[2,7] (VOUT); no longer PSU1.3 (OUT)
- new net +12V_FUSED_PSU1: D4.1 (K), F1.2, PSU1.1 (IN)
- new net 5V_PSU1_OUT: PSU1.3 (OUT), U5.6 (VIN2)
- new net Fan Controller Pico: HMI/I2C_SCL: CN2.7 (GPIO5)
- new net Fan Controller Pico: HMI/I2C_SDA: CN2.6 (GPIO4)
- new net V_{GS}_LIM: Q2.2 (GATE), R1.2, ZD1.2
- no-connect marks 21 -> 14
Other:
- sheet Fan Controller Pico: HMI ports: added 587_CTRL, ENCODER_A, ENCODER_B, GND, I2C_SCL, I2C_SDA, VSYS; removed none
- note added: "DESIGN SWITCHING: CALCULATED REQUIREMENTS"
- note added: "DMP3014SFDE"
- note added: "PWR INDICATOR"
- note added: "REF: texas instruments "fan controller overview""
- note added: "SIGNAL PULL-UP RESISTORS"
- note removed: "EFUSE INDICATOR"
- note removed: "TPS259482A"
- title: Raspberry Pi Pico Board Template -> Fan Controller TXU0204 Pico
- moved on the sheet: C3, C4, C5, C6, C7, CN1, D2, D3, FAN1, FAN2, FAN3, FAN4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

Commit message: tl;dr: update images, adjust rules, clean up notes, move 12v rail to power plane, adj signal traces
=======================================================================
added:
  misc/img/ - switch to 4-layer design from 2-layer
      2d-in1-cu.png
      2d-in2-cu.png

-----------------------------------------------------------------------
modified:
  ./ - adjusted rules, cleaned up signal trace routing
      fan-controller-txu0204-pico.kicad_dru
      fan-controller-txu0204-pico.kicad_pcb
      fan-controller-txu0204-pico.kicad_pro
      fan-controller-txu0204-pico.kicad_sch
  misc/img/ - update images
      2d-b-cu.png
      2d-f-cu.png
      schematic_fan1-fan2.png
      schematic_fan3-fan4.png
      schematic_overview.png
      schematic_pico-headers.png
      schematic_power-good-indicator.png
      schematic_power-supply-protection.png
Changed lines of the file:
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@@
 	(rectangle
 		(start 17.78 142.24)
-		(end 182.88 248.92)
+		(end 182.88 250.19)
 		(stroke
 			(width 0.1)
@@
 	(text "SIGNAL PULL-UP RESISTORS"
 		(exclude_from_sim no)
-		(at 425.45 177.8 0)
+		(at 425.45 260.2652 0)
 		(effects
 			(font
@@
 	(text_box "V_{CC} = 5V\nI_{OL} = 8mA\n\n8mA is the rec capacity, but\nmaybe should be limited to 5mA?\nlimit for TXU0204 drive capacity is\nlike 20 or 50mA, but maybe not OK\nfor fans\n\nR_{pullup(min)} = (V_{CC} - V_{outputlow(max)}) / I_{OL}\nR_{pullup(min)} = (5V - 3.33V) / 0.008A\n\nR_{pullup(min)} = 208.75Ω"
 		(exclude_from_sim no)
-		(at 425.45 177.8 0)
+		(at 425.45 260.2652 0)
 		(size 45.72 29.2948)
 		(margins 0.9525 0.9525 0.9525 0.9525)
@@
 		)
 	)
-	(text_box "pwm frequency\n~{             }\n\ndetermining what speeds are needed to support driving fans with PWM\n\"acceptable range\" for the PWM signal = 21kHz - 28kHz\ni think this is just arctic's quality control pass range\nperiod: https://www.firgelliauto.com/blogs/calculators/pwm-frequency-period-calculator\n25kHz (40us) to 28kHz (period 35.7us)\n40000ns to 357000ns???\n\nduty cycle usually is 0 rpm for the first like 5% up to 100%\nprobably just assume lowest is 1%\nso total period:\n25kHz (40.000 us) to 28kHz (period 35.714 us)\non time @1% duty cycle is 1/100 x period\n25kHz (0.4 us) to 28kHz (period 0.35714 us)\n400ns to 357ns?\n\nsrc: https://industrialmonitordirect.com/blogs/knowledgebase/calculating-maximum-pwm-frequency-for-mosfet-power-stages\nT = minimum Target pwm period\nf = frequency\nT_{PWM(min)} >= 357ns\nf_{PWM} = 28000Hz\n\nTXU0204\nV_{CCA} = 3.3V, V_{CCB} = 5V:\n(output enable / disable)\nt_{D(ON)} = 33ns max\nt_{D(OFF)} = 40ns max\n\nt_{rise} = 9ns?\nt_{fall} = 10ns????\n\nidk if this is the right way to calculate the time spent translating and saying that's the maximum theoretical pwm bandwidth\ni also don't think i'll even be enabling / disabling the devices for each pulse or anything; tachometer pulses aren't\ngoing to be switching the OE anyway\n\nunrealistic:\nt_{sw(total)} = t_{D(ON)} + T_{D(OFF)} + t_{rise} + t_{fall}\nt_{sw(total)} = 33ns + 40ns + 9ns + 10ns\nt_{sw(total)} = 92ns\nto ms for period/pwm frequency calculator:\nt_{sw(total)} = 0.000092ms\n10869.565kHz or 10.87MHz\n\nrealistic:\nt_{sw(total)} = t_{rise} + t_{fall}\nt_{sw(total)} = 9ns + 10ns\nt_{sw(total)} = 19ns\nto ms for period/pwm frequency calculator:\nt_{sw(total)} = 0.000019ms\n52631.579kHz or 52.63MHz\n\ntachometer readout\nmaximum acceptable noise level for a fan i am willing to be in the same room as\nN_{max} = 37dBa\nall fans will be 60mm or larger, and sanyo denki's lineup tops out at about 6k rpm if restricted to 60mm<= 37dBa>=\ntachometer is usually 2 pulses per rotation (because usually fan is 2 poles according to microchip)\nmy estimated limit of 9k rpm makes me wonder what the hell i had in my last case, because it probally exceeded 37dBa\nanyway\nhttps://www.analog.com/en/resources/design-notes/calculating-the-tachometer-register-value-of-the-max6615max6616.html\n(double-checking math)\n6k rpm tachometer = 12k pulses per minute\nf_{tach}Hz = 60cycles/min x 12000pulses/min\nf_{tach} = 720Hz\n\ni've got to be doing this all wrong, surely?\n\nhttps://calculator.academy/mbps-to-hz-calculator/\nassuming that it's 1 bit per channel\n\nB_{data} is data bandwidth in (mega) bits per second\nb_{channels} is bits transferred per cycle (number of active channels) ...in bits, believe it or not\nF_{bandwidth/channel} is frequency in Hz\n\nF_{bandwidth/channel}Hz = B_{data}Mbps / b_{channels}bits/Hz\nF_{bandwidth/channel}Hz = 200Mbps / 4bits/Hz\nF_{bandwidth/channel}Hz = 50MHz\n"
+	(text_box "pwm frequency\n~{             }\ndetermining what speeds are needed to support driving fans with PWM\n\"acceptable range\" for the PWM signal = 21kHz - 28kHz (i think this is just arctic's quality control range)\nperiod src: https://www.firgelliauto.com/blogs/calculators/pwm-frequency-period-calculator\n25kHz (period of 40us) to 28kHz (period of 35.7us)\n40000ns to 357000ns\n\nduty cycle usually is 0 rpm for the first like 5% up to 100%; just assuming lowest is 1%\nso total period:\n25kHz (period of 40.000 us) to 28kHz (period of 35.714 us)\non time @1% duty cycle is 1/100 x period\n	--> 25kHz (0.4 us) to 28kHz (period 0.35714 us)\n	--> 400ns to 357ns?\nsrc: https://industrialmonitordirect.com/blogs/knowledgebase/calculating-maximum-pwm-frequency-for-mosfet-power-stages\nT = minimum Target pwm period\nf = frequency\nT_{PWM(min)} >= 357ns\nf_{PWM} = 28000Hz\n\nTXU0204 translating V_{CCA} = 3.3V, V_{CCB} = 5V:\nt_{D(ON)} = 33ns max\nt_{D(OFF)} = 40ns max\nt_{rise} = 9ns?\nt_{fall} = 10ns????\n\nidk if this is the right way to calculate the time spent translating even be enabling / disabling the devices for each pulse\nunrealistic (toggling OE):\nt_{sw(total)} = t_{D(ON)} + T_{D(OFF)} + t_{rise} + t_{fall}\n	--> t_{sw(total)} = 33ns + 40ns + 9ns + 10ns\n	--> t_{sw(total)} = 92ns\nto ms for period/pwm frequency calculator:\nt_{sw(total)} = 0.000092ms\n	--> 10869.565kHz or 10.87MHz\n\nrealistic (not constantly toggling OE):\nt_{sw(total)} = t_{rise} + t_{fall}\n	--> t_{sw(total)} = 9ns + 10ns\n	--> t_{sw(total)} = 19ns\nto ms for period/pwm frequency calculator:\nt_{sw(total)} = 0.000019ms\n	--> 52631.579kHz or 52.63MHz\n\ntachometer readout:\nmaximum acceptable fan noise level\nN_{max} = 37dBa\nall fans will be 60mm or larger, and sanyo denki's lineup tops out at about 6k rpm if restricted to 60mm<= 37dBa>=\ntachometer is usually 2 pulses per rotation (because usually fan is 2 poles according to microchip)\nsrc: https://www.analog.com/en/resources/design-notes/calculating-the-tachometer-register-value-of-the-max6615max6616.html\n6k rpm tachometer = 12k pulses per minute\nf_{tach}Hz = 60cycles/min x 12000pulses/min\n	--> f_{tach} = 720Hz\ni've got to be doing this all wrong, surely?\n\nbit bandwidth to frequency conversion:\nsrc: https://calculator.academy/mbps-to-hz-calculator/\nassuming that it's 1 bit per channel\nB_{data} is data bandwidth in (mega) bits per second\nb_{channels} is bits transferred per cycle (number of active channels) ...in bits, believe it or not\nF_{bandwidth/channel} is frequency in Hz\n\nF_{bandwidth/channel}Hz = B_{data}Mbps / b_{channels}bits/Hz\n	--> F_{bandwidth/channel}Hz = 200Mbps / 4bits/Hz\n	--> F_{bandwidth/channel}Hz = 50MHz"
 		(exclude_from_sim no)
 		(at 425.45 2.54 0)
-		(size 110.49 169.889)
-		(margins 0.9525 0.9525 0.9525 0.9525)
-		(stroke
+		(size 113.03 138.43)
+		(margins 0.9525 0.9525 0.9525 0.9525)
+		(stroke

Commit message: tl;dr: re-added TVS protections to pwm and tach signals at fan connectors, rerouted 12v
========================================================================
added:
  misc/img/ - improved images for pcb etc
      fan-controller-txu0204-pico.svg
      fan-controller-txu0204-pico__Assembly.pdf
      fan-controller-txu0204-pico_color-b.svg
      fan-controller-txu0204-pico_color-f.svg
      fan-controller-txu0204-pico_color-in1.svg
      fan-controller-txu0204-pico_color-in2.svg

------------------------------------------------------------------------
removed:
  misc/img/ - restructured images of pcb
      2d-b-cu.png
      2d-b-cu_nocourtyards.png
      2d-f-cu.png
      2d-f-cu_nocourtyards.png
      2d-in1-cu.png
      2d-in2-cu.png

------------------------------------------------------------------------
modified:
  ./ - re-added TVS protections to tach and pwm signals at fan
    connectors, corrected some layout issues, rerouted 12vdc power to
    more effectively use the TVS diodes for the 12v power pins
      fan-controller-txu0204-pico.kicad_pcb
      fan-controller-txu0204-pico.kicad_pro
      fan-controller-txu0204-pico.kicad_sch

  misc/img/
      schematic_overview.png - re-added TVS protections to pwm and tach
Parts:
- added D10, D7, D8, D9: DF3A6.8FV, lsc-transistor:TRANS_SOT-723, symbol tvs-diodes-added:DF3A6.8FV_TOSHIBA
Connections:
- net GND: now also D10.3 (A), D7.3 (A), D8.3 (A), D9.3 (A)
- net PWM_FAN1: no longer TP9.1
- net PWM_FAN2: no longer TP10.1
- net PWM_FAN3: no longer TP13.1
- net PWM_FAN4: no longer TP14.1
- net TACH_FAN1: no longer TP11.1
- net TACH_FAN2: no longer TP12.1
- net TACH_FAN3: no longer TP15.1
- net TACH_FAN4: no longer TP16.1
- net at FAN3.3 (Pin_3), R12.1: now also TP15.1, D9.1 (K1)
- net at FAN2.4 (Pin_4), R16.1: now also TP12.1, D8.2 (K2)
- net at FAN3.4 (Pin_4), R17.1, R22.1: now also TP13.1, D9.2 (K2)
- net at FAN4.3 (Pin_3), R24.1, R26.1: now also TP14.1, D10.1 (K1)
- net at FAN4.4 (Pin_4), R18.1: now also TP16.1, D10.2 (K2)
- net at FAN1.3 (Pin_3), R11.1: now also TP11.1, D7.1 (K1)
- net at FAN2.3 (Pin_3), R23.1, R25.1: now also TP10.1, D8.1 (K1)
- net at FAN1.4 (Pin_4), R15.1, R21.1: now also TP9.1, D7.2 (K2)
Other:
- moved on the sheet: C3, C4, C5, C6, C7, CN1, D1, D4, F1, LD1, PSU1, Q1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
